File: hw/BigOleLCDBoard/BigOleLCDBoard.kicad_pcb (KiCad board)
At the start: 2 copper layers, 11 parts, among them J101 Conn_01x02, J102 Conn_01x04, J103 Conn_01x08, J104 Conn_01x08, U101 OD-103, U102 OD-103, U103 OD-103, U104 OD-103, U105 CY8CKIT-049-4XXX

Commit message: Ask WeMos D1-Mini, start layout
Parts:
- added H101: MountingHole, MountingHole:MountingHole_4.3mm_M4, F.Cu at (135.9, 21.6)
- added H102: MountingHole, MountingHole:MountingHole_4.3mm_M4, F.Cu at (135.9, 11.4)
- added H103: MountingHole, MountingHole:MountingHole_4.3mm_M4, F.Cu at (156.2, 11.4)
- added H104: MountingHole, MountingHole:MountingHole_4.3mm_M4, F.Cu at (146.0, 21.6)
- added H105: MountingHole, MountingHole:MountingHole_4.3mm_M4, F.Cu at (146.0, 11.4)
- added H106: MountingHole, MountingHole:MountingHole_4.3mm_M4, F.Cu at (156.2, 21.6)
- added U106: WeMos_D1_mini, Module:WEMOS_D1_mini_light, B.Cu at (107.5, 87.6)
- J101: value Conn_01x02 -> Conn_Power; moved to B.Cu
- J102: value Conn_01x04 -> Conn_i2c; moved to B.Cu
- J103, J104, R101, R102, U105: moved to B.Cu
- moved J102 32.7 mm to (9.53, 64.1)
- moved R101 28.5 mm to (11.2, 58.4), turned to 180 degrees
- moved R102 24.0 mm to (11.7, 53.3), turned to 0 degrees
- moved J103 7.65 mm to (25.4, 66.0)
- moved J104 7.59 mm to (17.8, 129.5)
- turned U105 to 0 degrees
Connections:
- U105 pad 11: unconnected-(U105-Pad11) -> Net-(U105-Pad11)
Routing:
- net /COM0: track 0.00 -> 341.5 mm, vias 0 -> 1
- net /COM2: track 0.00 -> 255.8 mm, vias 0 -> 2
- net (no net): track 0.00 -> 160.1 mm
- net /COM1: track 0.00 -> 142.0 mm
- net /COM3: track 0.00 -> 125.1 mm
- net /I2C_SCL: track 0.00 -> 110.5 mm
- net Net-(U101-Pad8): track 0.00 -> 105.7 mm
- net Net-(J103-Pad1): track 0.00 -> 105.3 mm
- net /I2C_SDA: track 0.00 -> 104.9 mm
- net Net-(U101-Pad7): track 0.00 -> 94.4 mm
- net Net-(U105-Pad11): track 0.00 -> 92.4 mm
- net Net-(U101-Pad6): track 0.00 -> 82.4 mm
- net Net-(U101-Pad9): track 0.00 -> 79.5 mm
- net Net-(U101-Pad4): track 0.00 -> 71.6 mm
- net Net-(U101-Pad3): track 0.00 -> 64.7 mm
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- added copper zone on F.Cu, net +3V3
- added copper zone on B.Cu, net GND
Other:
- board outline added: 337.8 x 132.1 mm
- board text added: "3v3 GND"
- board text added: "Power Via WeMos"
